File: LEOS-stack-template.kicad_sch (KiCad schematic)
At the start: 44 parts, among them J1 MicroFit_1x4, J2 MicroFit_1x4, U1 MCP2562FD, U2 MCP2518FD, U3 TPS55287, U4 MPM3620A, Y1 40 MHz

Commit message: mostly routed the vin to 12V buck converter
Parts:
- added J3: Conn_01x02_MountingPin, Connector_AMASS:AMASS_XT60IPW-M_1x03_P7.20mm_Horizontal, symbol Connector_Generic_MountingPin:Conn_01x02_MountingPin
- added J4, J5: Conn_01x02_Socket, Connector_JST:JST_XH_S2B-XH-A_1x02_P2.50mm_Horizontal, symbol Connector:Conn_01x02_Socket
- C_BOOT1: renamed from C04; footprint Capacitor_SMD:C_1206_3216Metric -> Capacitor_SMD:C_0805_2012Metric
- C_BOOT2: renamed from C05; footprint Capacitor_SMD:C_1206_3216Metric -> Capacitor_SMD:C_0805_2012Metric
- C_COMP1: renamed from C07; footprint Capacitor_SMD:C_1206_3216Metric -> Capacitor_SMD:C_0805_2012Metric
- C_COMP2: renamed from C06; footprint (none) -> Capacitor_SMD:C_0805_2012Metric
- C_SYNC1: renamed from C08; footprint (none) -> Capacitor_SMD:C_0805_2012Metric
- C_VCC1: renamed from C03; footprint Capacitor_SMD:C_1206_3216Metric -> Capacitor_SMD:C_0805_2012Metric
- C_in2: renamed from C01; footprint (none) -> Capacitor_SMD:C_0805_2012Metric
- C_out2: renamed from C02_1; footprint Capacitor_SMD:C_1206_3216Metric -> Capacitor_SMD:C_0805_2012Metric
- C_out3: renamed from C02_2; footprint Capacitor_SMD:C_1206_3216Metric -> Capacitor_SMD:C_0805_2012Metric
- renumbered R02 to R_CDC1, R3 to R_COMP1, R01 to R_FSW1, R04 to R_SNS1
Connections:
- net +12V: now also J4.1 (Pin_1)
- net +5V: now also J5.1 (Pin_1)
- net GND: now also J3.1 (Pin_1), J4.2 (Pin_2), J5.2 (Pin_2)
- net GNDA: now also C_COMP1.2, C_COMP2.2
- net VDC: now also J3.2 (Pin_2)
- no-connect marks 9 -> 10
