File: LEOS-power.kicad_pcb (KiCad board)
At the start: 2 copper layers, 100 x 100 mm, 22 parts, among them J1 MicroFit_1x4, J2 MicroFit_1x4, U1 MCP2562FD, U2 MCP2518FD, Y1 40 MHz

Commit message: Power board complete v1.0
Parts:
- added C_BOOT1: 0.1u, Capacitor_SMD:C_0603_1608Metric, F.Cu at (172.8, 110.5)
- added C_BOOT2: 0.1u, Capacitor_SMD:C_0603_1608Metric, F.Cu at (168.8, 110.5)
- added C_COMP1: 33n, Capacitor_SMD:C_0603_1608Metric, F.Cu at (161.3, 104.5)
- added C_COMP2: 15n, Capacitor_SMD:C_0603_1608Metric, F.Cu at (161.3, 107.0)
- added C_SYNC1: 47n, Capacitor_SMD:C_0603_1608Metric, F.Cu at (157.8, 102.0)
- added C_VCC1: 4.7u, Capacitor_SMD:C_0805_2012Metric, F.Cu at (165.3, 109.5)
- added C_in1: 10u, Capacitor_SMD:C_1206_3216Metric, F.Cu at (178.5, 105.0)
- added C_in2: 10u, Capacitor_SMD:C_1206_3216Metric, F.Cu at (181.2, 105.0)
- added C_in3: 10u, Capacitor_SMD:C_1206_3216Metric, F.Cu at (184.0, 105.0)
- added C_in4: 10u, Capacitor_SMD:C_1206_3216Metric, F.Cu at (186.8, 105.0)
- added C_out1: 22u, Capacitor_SMD:C_0805_2012Metric, F.Cu at (123.5, 90.0)
- added C_out2: 22u, Capacitor_SMD:C_0805_2012Metric, F.Cu at (169.8, 103.0)
- added C_out3: 22u, Capacitor_SMD:C_0805_2012Metric, F.Cu at (169.8, 100.5)
- added Cin1: 10u, Capacitor_SMD:C_0805_2012Metric, F.Cu at (126.9, 88.3)
- added J3: Power Input, LEOS:AMASS_XT60IPW-M_1x03_P7.20mm_Horizontal, F.Cu at (182.8, 90.7)
- added J4: 5V, Connector_JST:JST_XH_S2B-XH-A_1x02_P2.50mm_Horizontal, F.Cu at (189.8, 114.0)
- added J5: 5V, Connector_JST:JST_XH_S2B-XH-A_1x02_P2.50mm_Horizontal, F.Cu at (189.6, 123.0)
- added J6: 5V, Connector_JST:JST_XH_S2B-XH-A_1x02_P2.50mm_Horizontal, F.Cu at (189.6, 132.0)
- added J7: 12V, Connector_JST:JST_XH_S2B-XH-A_1x02_P2.50mm_Horizontal, F.Cu at (111.0, 111.0)
- added J8: 12V, Connector_JST:JST_XH_S2B-XH-A_1x02_P2.50mm_Horizontal, F.Cu at (111.3, 120.2)
- added J9: 12V, Connector_JST:JST_XH_S2B-XH-A_1x02_P2.50mm_Horizontal, F.Cu at (111.2, 130.1)
- added L1: 10u, LEOS:IND_TAIYO_NRS8030_TAY, F.Cu at (170.9, 117.0)
- added NT1: NetTie_2, NetTie:NetTie-2_SMD_Pad0.5mm, F.Cu at (163.8, 109.5)
- added R5: 100k, Resistor_SMD:R_0805_2012Metric_Pad1.20x1.40mm_HandSolder, F.Cu at (129.4, 85.8)
- added R6: 100k, Resistor_SMD:R_0805_2012Metric_Pad1.20x1.40mm_HandSolder, F.Cu at (126.9, 82.2)
- added R7: 19.1k, Resistor_SMD:R_0805_2012Metric_Pad1.20x1.40mm_HandSolder, F.Cu at (123.4, 83.2)
- added RBT1: 11k, Resistor_SMD:R_0805_2012Metric_Pad1.20x1.40mm_HandSolder, F.Cu at (157.8, 100.0)
- added RP1: 11k, Resistor_SMD:R_0805_2012Metric_Pad1.20x1.40mm_HandSolder, F.Cu at (134.5, 123.0)
- added RUP1: 100k, Resistor_SMD:R_0805_2012Metric_Pad1.20x1.40mm_HandSolder, F.Cu at (163.2, 102.0)
- added R_CDC1: 20k, Resistor_SMD:R_0805_2012Metric_Pad1.20x1.40mm_HandSolder, F.Cu at (160.2, 111.0)
- added R_COMP1: 7.5k, Resistor_SMD:R_0805_2012Metric_Pad1.20x1.40mm_HandSolder, F.Cu at (165.2, 107.0)
- added R_FSW1: 9.1k, Resistor_SMD:R_0805_2012Metric_Pad1.20x1.40mm_HandSolder, F.Cu at (177.0, 110.5)
- added R_SNS1: 16m, Resistor_SMD:R_0805_2012Metric_Pad1.20x1.40mm_HandSolder, F.Cu at (166.2, 101.0)
- added SW1: Pull Tag, LEOS:D2F-FL-A1, F.Cu at (122.0, 129.5)
- added SW2: Power Switch, Button_Switch_THT:SW_Slide_SPDT_Angled_CK_OS102011MA1Q, F.Cu at (129.1, 123.0)
- added TP5: 12V Test, TestPoint:TestPoint_Loop_D2.60mm_Drill0.9mm_Beaded, F.Cu at (156.4, 90.0)
- added TP6: GND Test Point, TestPoint:TestPoint_Loop_D2.60mm_Drill0.9mm_Beaded, F.Cu at (161.5, 90.0)
- added U3: TPS55287, LEOS:VQFN21_RYQ_TEX, F.Cu at (170.8, 107.0)
- added U4: MPM3620A, LEOS:IC18_MPM3620AGQV-Z_MNP, F.Cu at (122.9, 86.2)
Connections:
- A1 pad 11: unconnected-(A1-GPIO8-Pad11) -> /Power/SDA
- A1 pad 12: unconnected-(A1-GPIO9-Pad12) -> /Power/SCL
Routing:
- net +5V: track 107.8 -> 203.3 mm
- net /Power/EN: track 0.00 -> 76.0 mm, vias 0 -> 2
- net /Power/SCL: track 0.00 -> 57.8 mm, vias 0 -> 1
- net +12V: track 0.00 -> 57.4 mm
- net /Power/SDA: track 0.00 -> 53.7 mm, vias 0 -> 1
- net Net-(U3-VCC): track 0.00 -> 39.0 mm
- net GNDA: track 0.00 -> 30.8 mm, vias 0 -> 2
- net Net-(U3-DITH/SYNC): track 0.00 -> 17.2 mm, vias 0 -> 2
- net Net-(U3-FB/INT): track 0.00 -> 12.8 mm
- net Net-(U3-CDC): track 0.00 -> 11.3 mm, vias 0 -> 2
- net Net-(SW1-C): track 0.00 -> 8.60 mm
- net Net-(U3-FSW): track 0.00 -> 8.06 mm, vias 0 -> 2
- net Net-(U3-COMP): track 0.00 -> 6.88 mm
- net Net-(SW2-A): track 0.00 -> 6.48 mm
- net Net-(U4-EN): track 0.00 -> 4.37 mm
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- added copper zone on F.Cu, net +12V
- added copper zone on F.Cu, net /Power/FB
- added copper zone on F.Cu, net /Power/SW
- added copper zone on F.Cu, net GNDA
- added copper zone on F.Cu, net Net-(U3-ISP)
- added copper zone on F.Cu, net Net-(U3-SW1)
- added copper zone on F.Cu, net Net-(U3-SW2)
- added copper zone on F.Cu, net Net-(U3-VCC)
- added copper zone on F.Cu, net VDC
Other:
- board text added: "02/19/2026"
- board text added: "12V"
- board text added: "Input 12-24VDC"
- board text added: "LEOS Power Rev. 1"
- board text added: "OFF"
- board text added: "ON"
- board text added: "REMOVE BEFORE FLIGHT"
- board text removed: "LEOS CHANGE THIS NAME Rev. 3"

Commit message: v1.1 Fix UVLO and EN power source
Parts:
- added RP2: 100k, Resistor_SMD:R_0805_2012Metric, F.Cu at (136.5, 128.3)
- RP1: value 11k -> 750k; footprint Resistor_SMD:R_0805_2012Metric_Pad1.20x1.40mm_HandSolder -> Resistor_SMD:R_0805_2012Metric
- moved RP1 2.50 mm to (136.5, 124.5), turned to -90 degrees
Connections:
- RP1 pad 1: Net-(U3-VCC) -> VDC
Routing:
- net VDC: track 0.00 -> 66.3 mm
- net Net-(U3-VCC): track 39.0 -> 0.00 mm
- net Net-(SW2-A): track 6.48 -> 11.2 mm
Other:
- board text added: "02/20/2026"
- board text added: "LEOS Power Rev. 1.1"
- board text removed: "02/19/2026"
- board text removed: "LEOS Power Rev. 1"
